File: hardware/meshduino.sch (KiCad schematic (older format))
At the start: 10 parts, among them P1 mPCIe, P2 USB, U1 SM200, U2 FT232RL

Commit message: Remove external crystal since we're running at 5v
Parts:
- removed 12MHz1: CRYSTAL, Crystals:Crystal_HC49-SD_SMD, symbol CRYSTAL
Connections:
- wire segments 97 -> 91
- no-connect marks 50 -> 52
Changed lines of the file:
@@
 LIBS:valves
 LIBS:crumpschemes
-LIBS:stow-minipcie-single-cache
+LIBS:meshduino-cache
 EELAYER 25 0
 EELAYER END
@@
 	1    0    0    -1
 $EndComp
-Text GLabel 4500 4100 2    60   Input ~ 0
-FT_3v3
 Text GLabel 7550 3800 2    60   Output ~ 0
 RESET
@@
 	1    7050 5050
 	1    0    0    -1
-$EndComp
-$Comp
-L CRYSTAL 12MHz1
-U 1 1 55FA6B1E
-P 5150 3950
-F 0 "12MHz1" H 5150 4100 60  0000 C CNN
-F 1 "CRYSTAL" H 5150 3800 60  0000 C CNN
-F 2 "Crystals:Crystal_HC49-SD_SMD" H 5150 3950 60  0001 C CNN
-F 3 "" H 5150 3950 60  0000 C CNN
-	1    5150 3950
-	0    1    1    0
 $EndComp
 Text GLabel 5550 4500 0    60   Output ~ 0
@@
 	7050 4950 7050 5050
 Connection ~ 6900 4950
-Wire Wire Line
-	5150 3650 5450 3650
-Wire Wire Line
-	5450 3650 5450 3900
-Wire Wire Line
-	5450 3900 5650 3900
-Wire Wire Line
-	5150 4250 5450 4250
-Wire Wire Line
-	5450 4250 5450 4000
-Wire Wire Line
-	5450 4000 5650 4000
 Wire Wire Line
 	5650 4200 5650 4550
@@
 Wire Wire Line
 	6300 1950 6300 1900
-Connection ~ 5150 4250
-Connection ~ 5150 3650
+NoConn ~ 5650 3900
+NoConn ~ 5650 4000
 $EndSCHEMATC
